Commit message: created core URDF sim

File: src/articubot_one/description/robot_core.xacro (robot description, xacro)
@@ -1,4 +1,5 @@
 <?xml version="1.0"?>
 <robot xmlns:xacro="http://www.ros.org/wiki/xacro" >
+    <xacro:include filename="inertial_macros.xacro"/>
     <!-- COLOR MATERIAL -->
     <material name="white">
@@ -30,4 +31,13 @@
             <material name="white"/>
         </visual>
+        <collision>
+            <origin xyz="0.15 0 0.075"/>
+            <geometry>
+                <box size="0.3 0.3 0.15"/>
+            </geometry>
+        </collision>
+        <xacro:inertial_box mass="0.5" x="0.3" y="0.3" z="0.15">
+            <origin xyz="0.15 0 0.075" rpy="0 0 0"/>
+        </xacro:inertial_box>
     </link>
     <!-- LEFT WHEEL LINK -->
@@ -45,4 +55,12 @@
             <material name="blue"/>
         </visual>
+        <collision>
+            <geometry>
+                <cylinder radius="0.05" length="0.04"/>
+            </geometry>
+        </collision>
+        <xacro:inertial_cylinder mass="0.1" length="0.04" radius="0.05">
+            <origin xyz="0 0 0" rpy="0 0 0"/>
+        </xacro:inertial_cylinder>
     </link>
     <!-- RIGHT WHEEL LINK -->
@@ -60,4 +78,34 @@
             <material name="blue"/>
         </visual>
+        <collision>
+            <geometry>
+                <cylinder radius="0.05" length="0.04"/>
+            </geometry>
+        </collision>
+        <xacro:inertial_cylinder mass="0.1" length="0.04" radius="0.05">
+            <origin xyz="0 0 0" rpy="0 0 0"/>
+        </xacro:inertial_cylinder>
+    </link>
+    <!-- CASTER WHEEL LINK -->
+    <joint name="caster_wheel_joint" type="fixed">
+        <parent link="chassis"/>
+        <child link="caster_wheel"/>
+        <origin xyz="0.24 0 0"/>
+    </joint>
+    <link name="caster_wheel">
+        <visual>
+            <geometry>
+                <sphere radius="0.05"/>
+            </geometry>
+            <material name="black"/>
+        </visual>
+        <collision>
+            <geometry>
+                <sphere radius="0.05"/>
+            </geometry>
+        </collision>
+        <xacro:inertial_sphere mass="0.1" radius="0.05">
+            <origin xyz="0 0 0" rpy="0 0 0"/>
+        </xacro:inertial_sphere>
     </link>
 </robot>

Commit message: created base URDF simulation for lunabotics

File: src/articubot_one/description/robot_core.xacro (robot description, xacro)
@@ -21,5 +21,5 @@
         <parent link="base_link"/>
         <child link="chassis"/>
-        <origin xyz="-0.1 0 0 "/>
+        <origin xyz="-0.05 0 0 "/>
     </joint>
     <link name="chassis">
@@ -41,12 +41,38 @@
         </xacro:inertial_box>
     </link>
-    <!-- LEFT WHEEL LINK -->
-    <joint name="left_wheel_joint" type="continuous">
+    <!-- DIGGING LINK -->
+    <joint name="digging_joint" type="revolute">
         <parent link="base_link"/>
-        <child link="left_wheel"/>
+        <child link="digging_arm"/>
+        <origin xyz="0.25 0 0.05"/>
+        <axis xyz="0 1 0"/>
+        <limit lower="0" upper="1.5" effort="100.0" velocity="1.0"/>
+    </joint>
+    <link name="digging_arm">
+        <visual>
+            <origin xyz="0.1 0 0"/>
+            <geometry>
+                <box size="0.2 0.05 0.05"/>
+            </geometry>
+            <material name="white"/>
+        </visual>
+       <collision>
+            <origin xyz="0.1 0 0"/>
+            <geometry>
+                <box size="0.2 0.05 0.05"/>
+            </geometry>
+        </collision>
+        <xacro:inertial_box mass="0.3" x="0.2" y="0.05" z="0.05">
+            <origin xyz="0.15 0 0.075" rpy="0 0 0"/>
+        </xacro:inertial_box>
+    </link>
+    <!-- LEFT WHEEL LINK (BACK) -->
+    <joint name="left_back_wheel_joint" type="continuous">
+        <parent link="base_link"/>
+        <child link="left_back_wheel_front"/>
         <origin xyz="0 0.175 0" rpy="-${pi/2} 0 0 "/>
         <axis xyz="0 0 1"/>
     </joint>
-    <link name="left_wheel">
+    <link name="left_back_wheel_front">
         <visual>
             <geometry>
@@ -64,12 +90,12 @@
         </xacro:inertial_cylinder>
     </link>
-    <!-- RIGHT WHEEL LINK -->
-    <joint name="right_wheel_joint" type="continuous">
+    <!-- RIGHT WHEEL LINK (BACK) -->
+    <joint name="right_back_wheel_joint_front" type="continuous">
         <parent link="base_link"/>
-        <child link="right_wheel"/>
+        <child link="right_back_wheel_front"/>
         <origin xyz="0 -0.175 0" rpy="${pi/2} 0 0 "/>
         <axis xyz="0 0 -1"/>
     </joint>
-    <link name="right_wheel">
+    <link name="right_back_wheel_front">
         <visual>
             <geometry>
@@ -87,25 +113,49 @@
         </xacro:inertial_cylinder>
     </link>
-    <!-- CASTER WHEEL LINK -->
-    <joint name="caster_wheel_joint" type="fixed">
-        <parent link="chassis"/>
-        <child link="caster_wheel"/>
-        <origin xyz="0.24 0 0"/>
+    <!-- LEFT WHEEL LINK (FRONT) -->
+    <joint name="left_front_wheel_joint" type="continuous">
+        <parent link="base_link"/>
+        <child link="left_front_wheel"/>
+        <origin xyz="0.2 0.175 0" rpy="-${pi/2} 0 0 "/>
+        <axis xyz="0 0 1"/>
     </joint>
-    <link name="caster_wheel">
+    <link name="left_front_wheel">
         <visual>
             <geometry>
-                <sphere radius="0.05"/>
+                <cylinder radius="0.05" length="0.04"/>
             </geometry>
-            <material name="black"/>
+            <material name="blue"/>
         </visual>
         <collision>
             <geometry>
-                <sphere radius="0.05"/>
+                <cylinder radius="0.05" length="0.04"/>
             </geometry>
         </collision>
-        <xacro:inertial_sphere mass="0.1" radius="0.05">
+        <xacro:inertial_cylinder mass="0.1" length="0.04" radius="0.05">
             <origin xyz="0 0 0" rpy="0 0 0"/>
-        </xacro:inertial_sphere>
+        </xacro:inertial_cylinder>
+    </link>
+    <!-- RIGHT WHEEL LINK (FRONT) -->
+    <joint name="right_front_wheel_joint" type="continuous">
+        <parent link="base_link"/>
+        <child link="right_front_wheel"/>
+        <origin xyz="0.2 -0.175 0" rpy="${pi/2} 0 0 "/>
+        <axis xyz="0 0 -1"/>
+    </joint>
+    <link name="right_front_wheel">
+        <visual>
+            <geometry>
+                <cylinder radius="0.05" length="0.04"/>
+            </geometry>
+            <material name="blue"/>
+        </visual>
+        <collision>
+            <geometry>
+                <cylinder radius="0.05" length="0.04"/>
+            </geometry>
+        </collision>
+        <xacro:inertial_cylinder mass="0.1" length="0.04" radius="0.05">
+            <origin xyz="0 0 0" rpy="0 0 0"/>
+        </xacro:inertial_cylinder>
     </link>
 </robot>
