Commit message: added lidar to bot

File: src/articubot_one/description/gazebo_control.xacro (robot description, xacro)
@@ -3,5 +3,4 @@
     <gazebo>
         <plugin name="diff_drive" filename="libgazebo_ros_diff_drive.so">
-            <!-- ADD TO LUNABOTICS branch -->
             <!-- Wheel Info (Spacing and Dimensions) -->
             <left_joint>left_wheel_joint</left_joint>

File: src/articubot_one/description/robot.urdf.xacro (robot description, xacro)
@@ -3,4 +3,5 @@
     <xacro:include filename="robot_core.xacro" />
     <xacro:include filename="gazebo_control.xacro"/>
-    <!-- ADD TO LUNABOTICS -->
+    <xacro:include filename="lidar.xacro"/>
+    <xacro:include filename="camera.xacro"/>
 </robot>

File: src/articubot_one/description/robot_core.xacro (robot description, xacro)
@@ -2,8 +2,10 @@
 <robot xmlns:xacro="http://www.ros.org/wiki/xacro" >
     <xacro:include filename="inertial_macros.xacro"/>
-    <!-- ADD TO LUNABOTICS -->
     <!-- COLOR MATERIAL -->
     <material name="white">
         <color rgba="1 1 1 1" />
+    </material>
+    <material name="red">
+        <color rgba="1 0 0 1" />
     </material>
     <material name="orange">
