Commit message: added slam_toolbox package

File: src/articubot_one/description/lidar.xacro (robot description, xacro)
@@ -27,5 +27,5 @@
             <pose> 0 0 0 0 0 0 </pose>
             <!-- CHANGE TRUE OR FALSE -->
-            <visualize>false</visualize>
+            <visualize>true</visualize>
             <update_rate>10</update_rate>
             <ray>

File: src/articubot_one/description/robot_core.xacro (robot description, xacro)
@@ -20,4 +20,12 @@
     <!-- BASE LINK -->
     <link name="base_link"></link>
+    <!-- BASE FOOTPRINT LINK -->
+    <joint name="base_footprint_joint" type="fixed">
+        <parent link="base_link"/>
+        <child link="base_footprint"/>
+        <origin xyz="0 0 0" rpy="0 0 0"/>
+    </joint>
+    <link name="base_footprint">
+    </link>
     <!-- CHASSIS LINK -->
     <joint name="chassis_joint" type="fixed">
